File: power_distribution_board/power_distribution_board.sch (KiCad schematic (older format))
At the start: 67 parts, among them J1 CONN_01x03, J10 CONN_02X01, J11 CONN_02X01, J12 CONN_02X01, J13 CONN_02X01, J14 CONN_02X01, J15 CONN_02X01, J16 CONN_02X01, J17 CONN_02X01, J18 CONN_02X01, J19 CONN_02X01, J2 CONN_02X01, J20 CONN_02X01, J21 CONN_02X01, J22 CONN_02X01, J23 CONN_02X01, J3 CONN_02X01, J4 CONN_02X01, J5 CONN_02X01, J6 CONN_02X01, J7 CONN_02X01, J8 CONN_02X01, J9 CONN_02X01, Q1 NMOS_SSSGD, Q2 NMOS_SSSGD, Q3 NMOS_SSSGD, Q4 NMOS_SSSGD, Q5 Q_NMOS_GSD, U1 EHHD015A0A, U2 LTC1473, U3 EHHD010A0B, U4 LM317EMP, U5 BTS6133D, U6 A1120

Commit message: change inductor footprint; update order sheet
Parts:
- L1: footprint Inductors_SMD:L_0805 -> Inductors_SMD:L_1812
Changed lines of the file:
@@
 F 0 "L1" V 2150 6800 50  0000 C CNN
 F 1 "1m" V 2050 6800 50  0000 C CNN
-F 2 "Inductors_SMD:L_0805" H 2100 6800 50  0001 C CNN
+F 2 "Inductors_SMD:L_1812" H 2100 6800 50  0001 C CNN
 F 3 "" H 2100 6800 50  0001 C CNN
 	1    2100 6800
